Commit message: updated the ee to gripper offset in urdf

File: agents/iiwa14_with_fingers.urdf (robot description, URDF)
Before this commit: robot iiwa14, 76 links, 75 joints
Joints:
- joint iiwa_joint_gripper: origin xyz=0 0 0.16 rpy=0 0 0 -> xyz=0 0 0.180 rpy=0 0 0

File: agents/iiwa14_with_fingers_part_1_new.urdf (robot description, URDF)
Before this commit: robot iiwa14, 76 links, 75 joints
Joints:
- joint iiwa_joint_gripper: origin xyz=0 0 0.144 rpy=0 0 0 -> xyz=0 0 0.180 rpy=0 0 0
